File: KiCAD files - single PCB keyboard/Boston-keyboard-S.kicad_sch (KiCad schematic)
At the start: 578 parts, among them J705 TYPE-C-31-M12_13, J706 Conn_ARM_JTAG_SWD_10, Q701 DTC123J, Q702 AO4406AL, SW1 MXSwitch, SW10 MXSwitch, SW100 MXSwitch, SW101 MXSwitch, SW102 MXSwitch, SW103 MXSwitch, SW104 MXSwitch, SW105-1 MXSwitch, SW105-2 MXSwitch, SW106 MXSwitch, SW107 MXSwitch, SW108 MXSwitch, SW109 MXSwitch, SW11 MXSwitch, SW110 MXSwitch, SW111 MXSwitch, SW112 MXSwitch, SW113 MXSwitch, SW114 MXSwitch, SW115 MXSwitch, SW116 MXSwitch, SW117 MXSwitch, SW118 MXSwitch, SW119 MXSwitch, SW12 MXSwitch, SW120 MXSwitch, SW121 MXSwitch, SW122 MXSwitch, SW123 MXSwitch, SW124-1 MXSwitch, SW124-2 MXSwitch, SW125 MXSwitch, SW126 Rotary_Encoder_Switch_Chassis, SW127 MXSwitch, SW13 MXSwitch, SW14 MXSwitch, SW15 MXSwitch, SW16 MXSwitch, SW17 MXSwitch, SW18 MXSwitch, SW19 MXSwitch, SW2 MXSwitch, SW20 MXSwitch, SW200 SW_Push, SW21 MXSwitch, SW22 MXSwitch, SW23 MXSwitch, SW24 MXSwitch, SW25 MXSwitch, SW26 MXSwitch, SW27 MXSwitch, SW28 MXSwitch, SW29 MXSwitch, SW3 MXSwitch, SW30 MXSwitch, SW31 MXSwitch, SW32 MXSwitch, SW33 MXSwitch, SW34 MXSwitch, SW35 MXSwitch, SW36 MXSwitch, SW37 MXSwitch, SW38 MXSwitch, SW39 MXSwitch, SW4-1 MXSwitch, SW4-2 MXSwitch, SW40 MXSwitch, SW41 MXSwitch, SW42 MXSwitch, SW43 MXSwitch, SW44 MXSwitch, SW45 MXSwitch, SW46 MXSwitch, SW47 MXSwitch, SW48 MXSwitch, SW49 MXSwitch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

Commit message: Finalized layout
Parts:
- removed LOGO1: Logo_Open_Hardware_Large, acheronLogos:acheronShort_15.2x21mm, symbol Graphic:Logo_Open_Hardware_Large
- R710: value 33 -> 100
Connections:
- net RGBLED: now also U701.15 (PA5); no longer R710.2
- net at U705.4 (B): now also R710.2; no longer U1.6 (DIN)
- net at R710.1: now also U1.6 (DIN); no longer U701.15 (PA5)
Other:
- moved on the sheet: R710
Changed lines of the file:
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@@
     (stroke (width 0) (type solid) (color 0 0 0 0))
   )
-  (wire (pts (xy 364.49 372.11) (xy 364.49 388.62))
+  (wire (pts (xy 364.49 372.11) (xy 364.49 375.92))
+    (stroke (width 0) (type solid) (color 0 0 0 0))
+  )
+  (wire (pts (xy 364.49 383.54) (xy 364.49 388.62))
     (stroke (width 0) (type solid) (color 0 0 0 0))
   )
@@
     (stroke (width 0) (type solid) (color 0 0 0 0))
   )
-  (wire (pts (xy 883.92 233.68) (xy 897.89 233.68))
+  (wire (pts (xy 883.92 233.68) (xy 908.05 233.68))
     (stroke (width 0) (type solid) (color 0 0 0 0))
   )
@@
     (stroke (width 0) (type solid) (color 0 0 0 0))
   )
-  (wire (pts (xy 905.51 233.68) (xy 908.05 233.68))
-    (stroke (width 0) (type solid) (color 0 0 0 0))
-  )
   (wire (pts (xy 908.05 35.56) (xy 896.62 35.56))
     (stroke (width 0) (type solid) (color 0 0 0 0))
@@
     )
   )
+  (symbol (lib_id "Device:R") (at 364.49 379.73 180) (unit 1)
+    (in_bom yes) (on_board yes)
+    (property "Reference" "R710" (id 0) (at 361.95 382.27 90)
+      (effects (font (size 1.27 1.27)) (justify right))
+    )
+    (property "Value" "100" (id 1) (at 359.41 381 90)
+      (effects (font (size 1.27 1.27)) (justify right))
+    )
+    (property "Footprint" "Resistor_SMD:R_0805_2012Metric_Pad1.15x1.40mm_HandSolder" (id 2) (at 366.268 379.73 90)
+      (effects (font (size 1.27 1.27)) hide)
+    )
+    (property "Datasheet" "~" (id 3) (at 364.49 379.73 0)
+      (effects (font (size 1.27 1.27)) hide)
+    )
+  )
   (symbol (lib_id "Device:R") (at 364.49 412.75 0) (unit 1)
     (in_bom yes) (on_board yes)
@@
     )
   )
-  (symbol (lib_id "Device:R") (at 901.7 233.68 90) (unit 1)
-    (in_bom yes) (on_board yes)
-    (property "Reference" "R710" (id 0) (at 899.16 231.14 90)
-      (effects (font (size 1.27 1.27)) (justify right))
-    )
-    (property "Value" "33" (id 1) (at 900.43 228.6 90)
-      (effects (font (size 1.27 1.27)) (justify right))
-    )
-    (property "Footprint" "Resistor_SMD:R_0805_2012Metric_Pad1.15x1.40mm_HandSolder" (id 2) (at 901.7 235.458 90)
-      (effects (font (size 1.27 1.27)) hide)
-    )
-    (property "Datasheet" "~" (id 3) (at 901.7 233.68 0)
-      (effects (font (size 1.27 1.27)) hide)
-    )
-  )
   (symbol (lib_id "Device:R") (at 913.13 220.98 270) (unit 1)
     (in_bom yes) (on_board yes)
@@
     )
   )
-  (symbol (lib_id "Graphic:Logo_Open_Hardware_Large") (at 518.16 420.37 0) (unit 1)
-    (in_bom yes) (on_board yes)
-    (property "Reference" "LOGO1" (id 0) (at 518.16 407.67 0)
-      (effects (font (size 1.27 1.27)) hide)
-    )
-    (property "Value" "Logo_Open_Hardware_Large" (id 1) (at 518.16 430.53 0)
-      (effects (font (size 1.27 1.27)) hide)
-    )
-    (property "Footprint" "acheronLogos:acheronShort_15.2x21mm" (id 2) (at 518.16 420.37 0)
-      (effects (font (size 1.27 1.27)) hide)
-    )
-    (property "Datasheet" "~" (id 3) (at 518.16 420.37 0)
-      (effects (font (size 1.27 1.27)) hide)
-    )
-  )
   (symbol (lib_id "Graphic:Logo_Open_Hardware_Large") (at 518.16 444.5 0) (unit 1)
     (in_bom yes) (on_board yes)
@@
       (reference "LED90-2") (unit 1)
     )
-    (path "/00000000-0000-0000-0000-0000610b9a59"
-      (reference "LOGO1") (unit 1)
-    )
     (path "/00000000-0000-0000-0000-0000610bda06"
