File: Single PCB design/3D printed case- FR4 part files/Bottom/bottom/bottom.kicad_sch (KiCad schematic)
At the start: 13 parts

Commit message: Added more FR4 part files
Parts:
- removed H1, H10, H11, H12, H2, H3, H4, H5, H6, H7, H8, H9: MountingHole, MountingHole:MountingHole_3.2mm_M3_ISO7380, symbol Mechanical:MountingHole
- added H1, H10, H11, H12, H2, H3, H4, H5, H6, H7, H8, H9: MountingHole_Pad, MountingHole:MountingHole_3.2mm_M3_ISO7380_Pad, symbol Mechanical:MountingHole_Pad
- added HL2: MountingHole, BostonStreets:boston-streets-CU, symbol Mechanical:MountingHole
Connections:
- new net FrontCuFill: H1.1, H10.1, H11.1, H12.1, H2.1, H3.1, H4.1, H5.1, H6.1, H7.1, H8.1, H9.1
