File: Single PCB design/3D printed case- FR4 part files/Plate/FR4-plate/FR4-plate.kicad_pcb (KiCad board)
At the start: 2 copper layers, 396 x 161 mm, 11 parts

Commit message: Updated plate and bottom for 3D-printed case
Parts:
- added H12: MountingHole_Pad, MountingHole:MountingHole_2.5mm_Pad, F.Cu at (8.56, 52.7)
- added H13: MountingHole_Pad, MountingHole:MountingHole_2.5mm_Pad, F.Cu at (26.6, 19.4)
- added H14: MountingHole_Pad, MountingHole:MountingHole_2.5mm_Pad, F.Cu at (109.9, 14.7)
- added H15: MountingHole_Pad, MountingHole:MountingHole_2.5mm_Pad, F.Cu at (119.8, 52.7)
- added H16: MountingHole_Pad, MountingHole:MountingHole_2.5mm_Pad, F.Cu at (190.9, 14.7)
- added H17: MountingHole_Pad, MountingHole:MountingHole_2.5mm_Pad, F.Cu at (196.8, 52.7)
- added H18: MountingHole_Pad, MountingHole:MountingHole_2.5mm_Pad, F.Cu at (209.0, 52.7)
- added H19: MountingHole_Pad, MountingHole:MountingHole_2.5mm_Pad, F.Cu at (271.8, 14.7)
- added H20: MountingHole_Pad, MountingHole:MountingHole_2.5mm_Pad, F.Cu at (276.3, 52.7)
- added H21: MountingHole_Pad, MountingHole:MountingHole_2.5mm_Pad, F.Cu at (333.7, 14.7)
- added H22: MountingHole_Pad, MountingHole:MountingHole_2.5mm_Pad, F.Cu at (387.4, 52.7)
- added H23: MountingHole_Pad, MountingHole:MountingHole_2.5mm_Pad, F.Cu at (252.8, 149.5)
- added H24: MountingHole_Pad, MountingHole:MountingHole_2.5mm_Pad, F.Cu at (305.2, 119.1)
- added H25: MountingHole_Pad, MountingHole:MountingHole_2.5mm_Pad, F.Cu at (314.7, 149.5)
- added H26: MountingHole_Pad, MountingHole:MountingHole_5.3mm_M5_DIN965_Pad, F.Cu at (283.7, 52.7)
- added H27: MountingHole_Pad, MountingHole:MountingHole_5.3mm_M5_DIN965_Pad, F.Cu at (302.8, 52.7)
- added H28: MountingHole_Pad, MountingHole:MountingHole_5.3mm_M5_DIN965_Pad, F.Cu at (321.8, 52.7)
- added H29: MountingHole_Pad, MountingHole:MountingHole_5.3mm_M5_DIN965_Pad, F.Cu at (305.2, 126.6)
- moved H1 203.7 mm to (23.0, 5.38)
- moved H10 203.7 mm to (233.0, 157.2)
- moved H11 203.7 mm to (373.0, 157.2)
- moved H2 203.7 mm to (93.0, 5.38)
- moved H3 203.7 mm to (163.0, 5.38)
- moved H4 203.7 mm to (233.0, 5.38)
- moved H5 203.7 mm to (303.0, 5.38)
- moved H6 203.7 mm to (373.0, 5.38)
- moved H7 203.7 mm to (23.0, 157.2)
- moved H8 203.7 mm to (93.0, 157.2)
- moved H9 203.7 mm to (163.0, 157.2)
Routing:
- net Mounting-hole: vias 17 -> 0
Other:
- outline, holes or cut-outs redrawn
