File: Single PCB design/3D printed case- FR4 part files/Plate/FR4-plate/FR4-plate.kicad_sch (KiCad schematic)
At the start: 11 parts

Commit message: Updated plate and bottom for 3D-printed case
Parts:
- added H12, H13, H14, H15, H16, H17, H18, H19, H20, H21, H22, H23, H24, H25: MountingHole_Pad, MountingHole:MountingHole_2.5mm_Pad, symbol Mechanical:MountingHole_Pad
- added H26, H27, H28, H29: MountingHole_Pad, MountingHole:MountingHole_5.3mm_M5_DIN965_Pad, symbol Mechanical:MountingHole_Pad
Connections:
- net Mounting-hole: now also H12.1, H13.1, H14.1, H15.1, H16.1, H17.1, H18.1, H19.1, H20.1, H21.1, H22.1, H23.1, H24.1, H25.1, H26.1, H27.1, H28.1, H29.1
Other:
- note added: "4.7mm holes for PEM"
