File: Single PCB design/KiCAD files - single PCB keyboard/Boston-keyboard-S.kicad_sch (KiCad schematic)
At the start: 577 parts, among them J705 TYPE-C-31-M12_13, J706 Conn_ARM_JTAG_SWD_10, Q701 DTC123J, Q702 AO4406AL, SW1 MXSwitch, SW10 MXSwitch, SW100 MXSwitch, SW101 MXSwitch, SW102 MXSwitch, SW103 MXSwitch, SW104 MXSwitch, SW105-1 MXSwitch, SW105-2 MXSwitch, SW106 MXSwitch, SW107 MXSwitch, SW108 MXSwitch, SW109 MXSwitch, SW11 MXSwitch, SW110 MXSwitch, SW111 MXSwitch, SW112 MXSwitch, SW113 MXSwitch, SW114 MXSwitch, SW115 MXSwitch, SW116 MXSwitch, SW117 MXSwitch, SW118 MXSwitch, SW119 MXSwitch, SW12 MXSwitch, SW120 MXSwitch, SW121 MXSwitch, SW122 MXSwitch, SW123 MXSwitch, SW124-1 MXSwitch, SW124-2 MXSwitch, SW125 MXSwitch, SW126 Rotary_Encoder_Switch_Chassis, SW127 MXSwitch, SW13 MXSwitch, SW14 MXSwitch, SW15 MXSwitch, SW16 MXSwitch, SW17 MXSwitch, SW18 MXSwitch, SW19 MXSwitch, SW2 MXSwitch, SW20 MXSwitch, SW200 SW_Push, SW21 MXSwitch, SW22 MXSwitch, SW23 MXSwitch, SW24 MXSwitch, SW25 MXSwitch, SW26 MXSwitch, SW27 MXSwitch, SW28 MXSwitch, SW29 MXSwitch, SW3 MXSwitch, SW30 MXSwitch, SW31 MXSwitch, SW32 MXSwitch, SW33 MXSwitch, SW34 MXSwitch, SW35 MXSwitch, SW36 MXSwitch, SW37 MXSwitch, SW38 MXSwitch, SW39 MXSwitch, SW4-1 MXSwitch, SW4-2 MXSwitch, SW40 MXSwitch, SW41 MXSwitch, SW42 MXSwitch, SW43 MXSwitch, SW44 MXSwitch, SW45 MXSwitch, SW46 MXSwitch, SW47 MXSwitch, SW48 MXSwitch, SW49 MXSwitch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

Commit message: Updated RGBLED - pin 2 common anode instead of pin 1
Due to available RGB LEDs on JLCPCB
Parts:
- removed LED301: LED_ABRG, LED_THT:LED_D5.0mm-4_RGB, symbol Device:LED_ABRG
- added LED301: LED_RAGB, LED_THT:LED_D5.0mm-4_RGB, symbol Device:LED_RAGB
Connections:
- net +3V3: now also LED301.2 (A)
- net at U1.1 (OUTR): now also LED301.1 (RK)
- net at U1.2 (OUTG): now also LED301.3 (GK)
- net at U1.3 (OUTB): now also LED301.4 (BK)
