File: Single PCB design/KiCAD files - single PCB keyboard/Boston-keyboard-S.kicad_sch (KiCad schematic)
At the start: 598 parts, among them J701 Conn_01x02_Female, J702 Conn_01x03_Female, J705 TYPE-C-31-M12_13, J706 Conn_ARM_JTAG_SWD_10, Q701 DTC123J, Q702 AO4406AL, SW1 MXSwitch, SW10 MXSwitch, SW100 MXSwitch, SW101 MXSwitch, SW102 MXSwitch, SW103 MXSwitch, SW104 MXSwitch, SW105-1 MXSwitch, SW105-2 MXSwitch, SW106 MXSwitch, SW107 MXSwitch, SW108 MXSwitch, SW109 MXSwitch, SW11 MXSwitch, SW110 MXSwitch, SW111 MXSwitch, SW112 MXSwitch, SW113 MXSwitch, SW114 MXSwitch, SW115 MXSwitch, SW116 MXSwitch, SW117 MXSwitch, SW118 MXSwitch, SW119 MXSwitch, SW12 MXSwitch, SW120 MXSwitch, SW121 MXSwitch, SW122 MXSwitch, SW123 MXSwitch, SW124-1 MXSwitch, SW124-2 MXSwitch, SW125 MXSwitch, SW126 Rotary_Encoder_Switch_Chassis, SW127 MXSwitch, SW128 MXSwitch, SW129 MXSwitch, SW13 MXSwitch, SW14 MXSwitch, SW15 MXSwitch, SW16 MXSwitch, SW17 MXSwitch, SW18 MXSwitch, SW19 MXSwitch, SW2 MXSwitch, SW20-1 MXSwitch, SW20-2 MXSwitch, SW200 SW_Push, SW21 MXSwitch, SW22 MXSwitch, SW23 MXSwitch, SW24 MXSwitch, SW25 MXSwitch, SW26 MXSwitch, SW27 MXSwitch, SW28 MXSwitch, SW29 MXSwitch, SW3 MXSwitch, SW30 MXSwitch, SW31 MXSwitch, SW32 MXSwitch, SW33 MXSwitch, SW34 MXSwitch, SW35 MXSwitch, SW36 MXSwitch, SW37 MXSwitch, SW38 MXSwitch, SW39-1 MXSwitch, SW39-2 MXSwitch, SW39-3 MXSwitch, SW4-1 MXSwitch, SW4-2 MXSwitch, SW40 MXSwitch, SW41 MXSwitch, SW42 MXSwitch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

Commit message: Added ferrite to grounding wire
Parts:
- added L2: L_Core_Ferrite, Inductor_SMD:L_0805_2012Metric_Pad1.15x1.40mm_HandSolder, symbol Device:L_Core_Ferrite
Connections:
- net GND: now also L2.1; no longer H1.1
- new net: H1.1, L2.2
Changed lines of the file:
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@@
   (junction (at 1041.4 33.02) (diameter 0.3048) (color 0 0 0 0))
   (junction (at 1051.56 33.02) (diameter 0.3048) (color 0 0 0 0))
+  (no_connect (at 986.79 86.36))
   (no_connect (at 826.77 83.82))
-  (no_connect (at 986.79 83.82))
   (no_connect (at 826.77 86.36))
-  (no_connect (at 986.79 86.36))
+  (no_connect (at 986.79 83.82))
   (wire (pts (xy 19.05 326.39) (xy 27.94 326.39))
     (stroke (width 0) (type solid) (color 0 0 0 0))
@@
     (stroke (width 0) (type solid) (color 0 0 0 0))
   )
-  (wire (pts (xy 604.52 417.83) (xy 604.52 421.64))
+  (wire (pts (xy 604.52 425.45) (xy 604.52 429.895))
     (stroke (width 0) (type solid) (color 0 0 0 0))
   )
@@
     )
   )
-  (symbol (lib_id "power:GND") (at 604.52 421.64 0) (unit 1)
+  (symbol (lib_id "power:GND") (at 604.52 429.895 0) (unit 1)
     (in_bom yes) (on_board yes)
-    (property "Reference" "#PWR0110" (id 0) (at 604.52 427.99 0)
+    (property "Reference" "#PWR0110" (id 0) (at 604.52 436.245 0)
       (effects (font (size 1.27 1.27)) hide)
     )
-    (property "Value" "GND" (id 1) (at 604.647 426.0342 0))
-    (property "Footprint" "" (id 2) (at 604.52 421.64 0)
+    (property "Value" "GND" (id 1) (at 604.647 434.2892 0))
+    (property "Footprint" "" (id 2) (at 604.52 429.895 0)
       (effects (font (size 1.27 1.27)) hide)
     )
-    (property "Datasheet" "" (id 3) (at 604.52 421.64 0)
+    (property "Datasheet" "" (id 3) (at 604.52 429.895 0)
       (effects (font (size 1.27 1.27)) hide)
     )
@@
     )
   )
+  (symbol (lib_id "Device:L_Core_Ferrite") (at 604.52 421.64 180) (unit 1)
+    (in_bom yes) (on_board yes)
+    (property "Reference" "L2" (id 0) (at 595.63 421.64 90))
+    (property "Value" "L_Core_Ferrite" (id 1) (at 600.71 421.64 90))
+    (property "Footprint" "Inductor_SMD:L_0805_2012Metric_Pad1.15x1.40mm_HandSolder" (id 2) (at 604.52 421.64 0)
+      (effects (font (size 1.27 1.27)) hide)
+    )
+    (property "Datasheet" "~" (id 3) (at 604.52 421.64 0)
+      (effects (font (size 1.27 1.27)) hide)
+    )
+  )
   (symbol (lib_id "Device:L_Core_Ferrite") (at 803.91 102.87 0) (unit 1)
     (in_bom yes) (on_board yes)
@@
       (reference "L1") (unit 1) (value "L_Core_Ferrite") (footprint "Inductor_SMD:L_0805_2012Metric_Pad1.15x1.40mm_HandSolder")
     )
+    (path "/820a6847-2a2e-4a00-aacb-0787794a46e7"
+      (reference "L2") (unit 1) (value "L_Core_Ferrite") (footprint "Inductor_SMD:L_0805_2012Metric_Pad1.15x1.40mm_HandSolder")
+    )
     (path "/00000000-0000-0000-0000-00005ec88a29"
