File: Single PCB design/3D printed case- FR4 part files/Bottom/KiCAD - artwork on one side/bottom.kicad_sch (KiCad schematic)
At the start: 15 parts

Commit message: Updated bottom
Parts:
- removed H13: MountingHole_Pad, MountingHole:MountingHole_2.5mm_Pad, symbol Mechanical:MountingHole_Pad
Changed lines of the file:
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@@
   (junction (at 203.2 92.71) (diameter 0.3048) (color 0 0 0 0))
   (junction (at 203.2 99.06) (diameter 0.3048) (color 0 0 0 0))
-  (junction (at 234.95 92.71) (diameter 0.3048) (color 0 0 0 0))
   (wire (pts (xy 116.84 92.71) (xy 118.11 92.71))
     (stroke (width 0) (type solid) (color 0 0 0 0))
@@
     (stroke (width 0) (type solid) (color 0 0 0 0))
   )
-  (wire (pts (xy 234.95 86.36) (xy 234.95 92.71))
-    (stroke (width 0) (type solid) (color 0 0 0 0))
-  )
-  (wire (pts (xy 234.95 92.71) (xy 234.95 97.79))
+  (wire (pts (xy 234.95 86.36) (xy 234.95 97.79))
     (stroke (width 0) (type solid) (color 0 0 0 0))
   )
@@
     )
     (property "Datasheet" "~" (id 3) (at 205.74 105.41 0)
-      (effects (font (size 1.27 1.27)) hide)
-    )
-  )
-  (symbol (lib_id "Mechanical:MountingHole_Pad") (at 237.49 92.71 270) (unit 1)
-    (in_bom yes) (on_board yes)
-    (property "Reference" "H13" (id 0) (at 242.57 91.44 90)
-      (effects (font (size 1.27 1.27)) (justify left))
-    )
-    (property "Value" "MountingHole_Pad" (id 1) (at 242.57 92.71 90)
-      (effects (font (size 1.27 1.27)) (justify left))
-    )
-    (property "Footprint" "MountingHole:MountingHole_2.5mm_Pad" (id 2) (at 237.49 92.71 0)
-      (effects (font (size 1.27 1.27)) hide)
-    )
-    (property "Datasheet" "~" (id 3) (at 237.49 92.71 0)
       (effects (font (size 1.27 1.27)) hide)
     )
@@
       (reference "H12") (unit 1)
     )
-    (path "/63c0377d-5da0-46e0-8b20-29746cf47d80"
-      (reference "H13") (unit 1)
-    )
     (path "/587302cf-ab79-45d3-8d0c-f3b140adfffc"
