File: Single PCB design/3D printed case- FR4 part files/Plate/Current FR4 plate/FR4-plate-new.kicad_pcb (KiCad board)
At the start: 2 copper layers, 396 x 161 mm, 29 parts

Commit message: Updated bottom
Other:
- outline, holes or cut-outs redrawn
- board text added: "1.25u"
- board text added: "1.25u Alt"
- board text added: "1.25u Ctrl"
- board text added: "1.25u Win"
- board text added: "1.5u Alt"
- board text added: "1.5u Ctrl"
- board text added: "1u Alt"
- board text added: "1u Ctrl"
- board text added: "6.25u"
- board text added: "7u"
- board text added: "JLCJLCJLCJLC"
- board text added: "Test your bottom row by installing keycaps before soldering switches!"

Commit message: Fixed silkcreen on FR4 plate
Other:
- outline, holes or cut-outs redrawn
- board text removed: "1.25u Alt"
