File: Boston - Current design/3D-printed case - parts/Plate/Current FR4 plate (split space support)/FR4-plate-new.kicad_pcb (KiCad board)
At the start: 2 copper layers, 396 x 161 mm, 29 parts

Commit message: Tightened up clearances on M2 holes, added solder mask back onto the bottom layer
Parts:
- H12, H13, H14, H15, H16, H17, H18, H19, H20, H21, H22, H23, H24, H25: footprint MountingHole:MountingHole_2.5mm_Pad -> MountingHole:MountingHole_2.2mm_M2_Pad
