File: Boston - Current design/KiCAD files - PCB/Boston-keyboard-S.kicad_sch (KiCad schematic)
At the start: 599 parts, among them J701 Conn_01x02_Female, J702 Conn_01x03_Female, J705 TYPE-C-31-M12_13, J706 Conn_ARM_JTAG_SWD_10, Q701 DTC123J, Q702 AO4406AL, SW1 MXSwitch, SW10 MXSwitch, SW100 MXSwitch, SW101 MXSwitch, SW102 MXSwitch, SW103 MXSwitch, SW104 MXSwitch, SW105-1 MXSwitch, SW105-2 MXSwitch, SW106 MXSwitch, SW107 MXSwitch, SW108 MXSwitch, SW109 MXSwitch, SW11 MXSwitch, SW110 MXSwitch, SW111 MXSwitch, SW112 MXSwitch, SW113 MXSwitch, SW114 MXSwitch, SW115 MXSwitch, SW116 MXSwitch, SW117 MXSwitch, SW118 MXSwitch, SW119 MXSwitch, SW12 MXSwitch, SW120 MXSwitch, SW121 MXSwitch, SW122 MXSwitch, SW123 MXSwitch, SW124-1 MXSwitch, SW124-2 MXSwitch, SW125 MXSwitch, SW126 Rotary_Encoder_Switch_Chassis, SW127 MXSwitch, SW128 MXSwitch, SW129 MXSwitch, SW13 MXSwitch, SW14 MXSwitch, SW15 MXSwitch, SW16 MXSwitch, SW17 MXSwitch, SW18 MXSwitch, SW19 MXSwitch, SW2 MXSwitch, SW20-1 MXSwitch, SW20-2 MXSwitch, SW200 SW_Push, SW21 MXSwitch, SW22 MXSwitch, SW23 MXSwitch, SW24 MXSwitch, SW25 MXSwitch, SW26 MXSwitch, SW27 MXSwitch, SW28 MXSwitch, SW29 MXSwitch, SW3 MXSwitch, SW30 MXSwitch, SW31 MXSwitch, SW32 MXSwitch, SW33 MXSwitch, SW34 MXSwitch, SW35 MXSwitch, SW36 MXSwitch, SW37 MXSwitch, SW38 MXSwitch, SW39-1 MXSwitch, SW39-2 MXSwitch, SW39-3 MXSwitch, SW4-1 MXSwitch, SW4-2 MXSwitch, SW40 MXSwitch, SW41 MXSwitch, SW42 MXSwitch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

Commit message: Cleaned up a bunch of files
Parts:
- F701: value Polyfuse -> 1.5A Polyfuse
Changed lines of the file:
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@@
   (junction (at 815.34 153.67) (diameter 0.3048) (color 0 0 0 0))
   (junction (at 825.5 153.67) (diameter 0.3048) (color 0 0 0 0))
-  (no_connect (at 739.14 85.725))
   (no_connect (at 739.14 88.265))
-  (no_connect (at 536.575 505.46))
+  (no_connect (at 739.14 85.725))
   (no_connect (at 536.575 502.92))
+  (no_connect (at 536.575 505.46))
   (wire (pts (xy 19.05 326.39) (xy 27.94 326.39))
     (stroke (width 0) (type solid) (color 0 0 0 0))
@@
     (in_bom yes) (on_board yes)
     (property "Reference" "F701" (id 0) (at 712.47 142.875 90))
-    (property "Value" "Polyfuse" (id 1) (at 712.47 145.1864 90))
+    (property "Value" "1.5A Polyfuse" (id 1) (at 712.47 145.1864 90))
     (property "Footprint" "Fuse:Fuse_1812_4532Metric_Pad1.30x3.40mm_HandSolder" (id 2) (at 707.39 149.86 0)
       (effects (font (size 1.27 1.27)) (justify left) hide)
@@
     )
     (path "/00000000-0000-0000-0000-00005dd252e1"
-      (reference "F701") (unit 1) (value "Polyfuse") (footprint "Fuse:Fuse_1812_4532Metric_Pad1.30x3.40mm_HandSolder")
+      (reference "F701") (unit 1) (value "1.5A Polyfuse") (footprint "Fuse:Fuse_1812_4532Metric_Pad1.30x3.40mm_HandSolder")
     )
     (path "/d4e35a86-b7af-44fe-a5dc-9f8d7b05c959"
